File: midi-vidi.brd (EAGLE design)
At the start: 152.5 x 43.6 mm, 80 parts, among them IC1 74HC595D, IC2 74HC595D, IC3 4051D, IC4 REG1117

Commit message: updates
Parts:
- removed C12: (no value), rcl:E2,5-6E
- removed R17: (no value), rcl:R0805
- removed U$12: MAX4311SO14, jason_eagle6:SO14
- removed U$14: PIC16F1825SO14, jasons_stuff:SO14
- added C10, C9: (no value), rcl:E2,5-6E
- added IC6: REG1117, burr-brown:SOT223
- added IC7: 74HC595D, 74xx-eu:SO16
- added L1: (no value), wuerth-elektronik:WE-TI_L
- added RR17: (no value), rcl:R0805
- IC1: value 74HC595D -> MAX4311SO14; device 74xx-eu:SO16 -> jason_eagle6:SO14
- IC2: value 74HC595D -> PIC16F1825SO14; device 74xx-eu:SO16 -> jasons_stuff:SO14
- IC3: value 4051D -> 74HC595D; device 40xx:SO16 -> 74xx-eu:SO16
- IC4: value REG1117 -> 4051D; device burr-brown:SOT223 -> 40xx:SO16
- moved R21 119.5 mm to (21.6, 39.4), turned to 90 degrees
- moved R6 99.1 mm to (146.2, 16.5), turned to 0 degrees
- moved R20 96.8 mm to (30.5, 32.0), turned to 90 degrees
- moved R28 96.2 mm to (33.4, 8.64), turned to 180 degrees
- moved R19 86.4 mm to (30.5, 38.1), turned to 270 degrees
- moved R4 79.5 mm to (112.5, 30.5)
- moved R27 78.2 mm to (46.0, 8.51), turned to 180 degrees
- moved R7 78.0 mm to (133.3, 16.5)
- moved R3 70.3 mm to (116.1, 29.5), turned to 90 degrees
- moved C1 66.0 mm to (130.8, 26.7)
- moved R2 62.9 mm to (119.4, 35.6), turned to 270 degrees
- moved R15 62.7 mm to (80.0, 16.5), turned to 0 degrees
- moved R5 61.8 mm to (112.5, 27.9), turned to 180 degrees
- moved R18 55.7 mm to (48.3, 31.8), turned to 270 degrees
- moved IC2 50.9 mm to (91.4, 31.8)
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- renumbered B1 to IC8, J1 to ICSP, L10 to LED1, L11 to LED2, L2 to LED9, L3 to LED10, L4 to LED8, L5 to LED7, L6 to LED6, L7 to LED5, L8 to LED4, L9 to LED3, S2 to SW7, S3 to SW6, S4 to SW8, S5 to SW5, S6 to SW4, S7 to SW1, S8 to SW2, S9 to SW3, U$13 to IC5, U$5 to D1
Connections:
- new net N$15: C10.+, C7.2, IC6.3, L1.1
- net A0A: now also IC7.5; no longer IC2.5
- net A0B: now also IC1.2, IC7.6; no longer IC2.6, U$12.2
- net A1A: now also IC7.4; no longer IC2.4
- net A1B: now also IC1.1, IC7.7; no longer IC2.7, U$12.1
- net AD0: now also IC2.8, IC4.11; no longer IC3.11, U$14.8
- net AD1: now also IC2.9, IC4.10; no longer IC3.10, U$14.9
- net AD2: now also IC2.10, IC4.9; no longer IC3.9, U$14.10
- net DAT: now also IC2.12, IC3.14; no longer IC1.14, U$14.12
- net GND: now also C10.-, C2.1, C4.1, C5.2, C6.2, C9.-, IC1.11, IC2.14, IC3.13, IC4.6, IC4.7, IC4.8, IC6.1, IC7.13, IC7.8, R15.1, R18.1, R20.1, R22.1, R23.1, R24.1, R5.1, R7.1; no longer C12.-, C2.2, C4.2, C5.1, C6.1, IC1.13, IC1.8, IC2.13, IC2.8, IC3.6, IC3.7, IC4.1, R1.1, R10.1, R11.1, R13.1, R17.1, R27.1, R3.1, R4.1, U$12.11, U$14.14
- net IN: now also IC2.11, IC4.3, R14.1; no longer IC3.3, R26.1, U$14.11
- net MIDI: now also IC2.5, R19.2; no longer R16.2, U$14.5
- net N$1: now also R24.2; no longer R4.2
- net N$10: now also IC1.7, R7.2; no longer R9.2, U$12.7
- net N$11: now also IC1.8, R8.2; no longer R10.2, U$12.8
- net N$12: now also IC1.5, R6.2; no longer R8.2, U$12.5
- net N$13: now also IC1.14, R3.2, R4.2; no longer R12.2, R14.2, U$12.14
- net N$14: now also IC1.13, R3.1, R5.2; no longer R12.1, R13.2, U$12.13
- net N$16: now also R4.1; no longer R14.1
- net N$17: now also IC1.10, R9.2; no longer R11.2, U$12.10
- net N$19: now also R10.2; no longer R21.2
- net N$2: now also R23.2; no longer R3.2
- net N$20: now also R11.2; no longer R20.2
- net N$21: now also R12.2; no longer R19.2
- net N$22: now also R20.2; no longer R17.2
- net N$23: now also IC3.15, R10.1; no longer IC1.15, R21.1
- net N$24: now also R13.2; no longer R18.2
- net N$25: now also IC3.1, R11.1; no longer IC1.1, R20.1
- net N$26: now also IC3.2, R12.1; no longer IC1.2, R19.1
- net N$27: now also IC3.3, R13.1; no longer IC1.3, R18.1
- net N$28: now also IC3.4; no longer IC1.4
- net N$29: now also IC3.5, R26.1; no longer IC1.5, R24.1
- net N$3: now also R22.2; no longer R2.2
- net N$30: now also IC3.6, R28.1; no longer IC1.6, R23.1
- net N$31: now also IC3.7, R27.1; no longer IC1.7, R22.1
- net N$33: now also R26.2; no longer R24.2
- net N$34: now also R28.2; no longer R23.2
- net N$35: now also R27.2; no longer R22.2
- net N$36: now also R2.2; no longer R27.2
- net N$37: now also IC4.4; no longer IC3.4
- net N$38: now also IC4.2; no longer IC3.2
- net N$39: now also IC4.5; no longer IC3.5
- net N$4: now also R15.2; no longer R1.2
- net N$40: now also IC4.1; no longer IC3.1
- net N$41: now also IC4.12; no longer IC3.12
- net N$42: now also IC4.15; no longer IC3.15
- net N$43: now also IC4.14; no longer IC3.14
- net N$44: now also IC4.13; no longer IC3.13
- net N$45: now also IC2.13; no longer U$14.13
- net N$47: now also IC3.9, IC7.14; no longer IC1.9, IC2.14
- net N$48: now also IC2.4; no longer U$14.4
- net N$5: now also R16.2, RR17.2; no longer R5.2, R7.2
- net N$50: now also R1.2; no longer R28.2
- net N$51: now also L1.2; no longer C7.2, IC4.3
- net N$6: now also R18.2, RR17.1; no longer R5.1, R6.2
- net N$7: now also R16.1; no longer R7.1
- net N$8: now also R21.1; no longer R15.1
- net N$9: now also R21.2; no longer R15.2
- net NSHDNA: now also IC2.6; no longer U$14.6
- net NSHDNB: now also IC1.12, IC2.7; no longer U$12.12, U$14.7
- net SH_CLK: now also IC2.3, IC3.11, IC7.11; no longer IC1.11, IC2.11, U$14.3
- net ST_CLK: now also IC2.2, IC3.10, IC7.10; no longer IC1.10, IC2.10, U$14.2
- net VCC: now also C2.2, C4.2, C5.1, C6.1, C9.+, IC1.4, IC2.1, IC3.12, IC4.16, IC6.2, IC7.12, IC7.16, R1.1, R14.2, R19.1; no longer C12.+, C2.1, C4.1, C5.2, C6.2, IC1.12, IC1.16, IC2.12, IC2.16, IC4.2, R16.1, R26.2, R28.1, U$12.4, U$14.1
Routing:
- net GND: track 8.80 -> 36.7 mm
- net N$15: track 0.00 -> 15.6 mm
- net N$51: track 89.8 -> 77.1 mm
- net N$37: track 42.6 -> 49.1 mm
- net N$43: track 34.3 -> 40.9 mm
- net N$42: track 45.6 -> 52.1 mm
- net N$44: track 22.9 -> 29.4 mm
- net N$40: track 22.4 -> 28.9 mm
- net N$39: track 53.9 -> 60.4 mm
- net N$38: track 32.4 -> 38.9 mm
- net N$41: track 12.2 -> 18.7 mm
- net VCC: track 239.0 -> 245.4 mm, vias 6 -> 8
- net A1B: track 105.4 -> 103.2 mm
- net A0B: track 102.7 -> 100.5 mm
- net N$46: track 10.0 -> 12.2 mm
