File: midi-vidi.sch (EAGLE design)
At the start: 80 parts, among them IC1 74HC595D, IC2 74HC595D, IC3 4051D, IC4 REG1117

Commit message: updates
Parts:
- removed C12: (no value), rcl:CPOL-EUE2,5-6E
- removed J1: (no value), tag-connect:TC2030-MCP-NL
- removed L2, L3: (no value), led:LED3MM
- removed R17: (no value), rcl:R-EU_R0805
- removed U$12, U$13: MAX4311SO14, jason_eagle6:MAX4311SO14
- removed U$14: PIC16F1825SO14, jasons_stuff:PIC16F1825SO14
- added C10, C9: (no value), rcl:CPOL-EUE2,5-6E
- added IC5: MAX4311SO14, jason_eagle6:MAX4311SO14
- added IC6: REG1117, burr-brown:REG1117
- added IC7: 74HC595D, 74xx-eu:74HC595D
- added ICSP: (no value), tag-connect:TC2030-MCP-NL
- added L1: (no value), wuerth-elektronik:WE-TI_L
- added LED10, LED9: (no value), led:LED3MM
- added RR17: (no value), rcl:R-EU_R0805
- IC1: value 74HC595D -> MAX4311SO14; device 74xx-eu:74HC595D -> jason_eagle6:MAX4311SO14
- IC2: value 74HC595D -> PIC16F1825SO14; device 74xx-eu:74HC595D -> jasons_stuff:PIC16F1825SO14
- IC3: value 4051D -> 74HC595D; device 40xx:4051D -> 74xx-eu:74HC595D
- IC4: value REG1117 -> 4051D; device burr-brown:REG1117 -> 40xx:4051D
- renumbered B1 to IC8, L10 to LED1, L11 to LED2, L4 to LED8, L5 to LED7, L6 to LED6, L7 to LED5, L8 to LED4, L9 to LED3, S2 to SW7, S3 to SW6, S4 to SW8, S5 to SW5, S6 to SW4, S7 to SW1, S8 to SW2, S9 to SW3, U$5 to D1
Connections:
- new net N$15: C10.+, C7.2, IC6.VIN, L1.2
- net A0A: now also IC5.A0, IC7A.QF; no longer IC2A.QF, U$13.A0
- net A0B: now also IC1.A0, IC7A.QG; no longer IC2A.QG, U$12.A0
- net A1A: now also IC5.A1, IC7A.QE; no longer IC2A.QE, U$13.A1
- net A1B: now also IC1.A1, IC7A.QH; no longer IC2A.QH, U$12.A1
- net AD0: now also IC2.RC2, IC4A.A; no longer IC3A.A, U$14.RC2
- net AD1: now also IC2.RC1/SDA/SDI, IC4A.B; no longer IC3A.B, U$14.RC1/SDA/SDI
- net AD2: now also IC2.RCO/SCL/SCK, IC4A.C; no longer IC3A.C, U$14.RCO/SCL/SCK
- net DAT: now also IC2.RA1/ICPCLK, IC3A.SER, ICSP.ICSP_CLK/PGC; no longer IC1A.SER, J1.ICSP_CLK/PGC, U$14.RA1/ICPCLK
- net GND: now also C10.-, C2.1, C4.1, C5.2, C6.2, C9.-, IC1.VEE, IC2.VSS, IC3A.G, IC4A.INH, IC4P.GND, IC4P.VEE, IC5.VEE, IC6.GND, IC7A.G, IC7P.GND, ICSP.VSS(GND), LED10.C, R15.1, R18.1, R20.1, R22.1, R23.1, R24.1, R5.1, R7.1; no longer C12.-, C2.2, C4.2, C5.1, C6.1, IC1A.G, IC1P.GND, IC2A.G, IC2P.GND, IC3A.INH, IC3P.VEE, IC4.GND, J1.VSS(GND), L3.C, R1.1, R10.1, R11.1, R13.1, R17.1, R27.1, R3.1, R4.1, U$12.VEE, U$13.VEE, U$14.VSS
- net IN: now also IC2.RA2/INT, IC4A.X, R14.1; no longer IC3A.X, R26.1, U$14.RA2/INT
- net MIDI: now also IC2.RC5/RX, R19.2; no longer R16.2, U$14.RC5/RX
- net N$1: now also IC5.IN3, R24.2; no longer R4.2, U$13.IN3
- net N$10: now also IC1.IN1, R7.2; no longer R9.2, U$12.IN1
- net N$11: now also IC1.IN2, R8.2; no longer R10.2, U$12.IN2
- net N$12: now also IC1.IN0, R6.2; no longer R8.2, U$12.IN0
- net N$13: now also IC1.OUT, R3.2, R4.2; no longer R12.2, R14.2, U$12.OUT
- net N$14: now also IC1.FB, R3.1, R5.2; no longer R12.1, R13.2, U$12.FB
- net N$16: now also R4.1; no longer R14.1
- net N$17: now also IC1.IN3, R9.2; no longer R11.2, U$12.IN3
- net N$19: now also R10.2; no longer R21.2
- net N$2: now also IC5.IN2, R23.2; no longer R3.2, U$13.IN2
- net N$20: now also R11.2; no longer R20.2
- net N$21: now also R12.2; no longer R19.2
- net N$22: now also R20.2; no longer R17.2
- net N$23: now also IC3A.QA, R10.1; no longer IC1A.QA, R21.1
- net N$24: now also R13.2; no longer R18.2
- net N$25: now also IC3A.QB, R11.1; no longer IC1A.QB, R20.1
- net N$26: now also IC3A.QC, R12.1; no longer IC1A.QC, R19.1
- net N$27: now also IC3A.QD, R13.1; no longer IC1A.QD, R18.1
- net N$28: now also IC3A.QE; no longer IC1A.QE
- net N$29: now also IC3A.QF, R26.1; no longer IC1A.QF, R24.1
- net N$3: now also IC5.IN1, R22.2; no longer R2.2, U$13.IN1
- net N$30: now also IC3A.QG, R28.1; no longer IC1A.QG, R23.1
- net N$31: now also IC3A.QH, R27.1; no longer IC1A.QH, R22.1
- net N$33: now also R26.2; no longer R24.2
- net N$34: now also R28.2; no longer R23.2
- net N$35: now also R27.2; no longer R22.2
- net N$36: now also LED9.C, R2.2; no longer L2.C, R27.2
- net N$37: now also IC4A.X7; no longer IC3A.X7
- net N$38: now also IC4A.X6; no longer IC3A.X6
- net N$39: now also IC4A.X5; no longer IC3A.X5
- net N$4: now also IC5.IN0, R15.2; no longer R1.2, U$13.IN0
- net N$40: now also IC4A.X4; no longer IC3A.X4
- net N$41: now also IC4A.X3; no longer IC3A.X3
- net N$42: now also IC4A.X2; no longer IC3A.X2
- net N$43: now also IC4A.X1; no longer IC3A.X1
- net N$44: now also IC4A.X0; no longer IC3A.X0
- net N$45: now also IC2.RA0/ICSPDAT, ICSP.ICSP_DAT/PGD, LED9.A; no longer J1.ICSP_DAT/PGD, L2.A, U$14.RA0/ICSPDAT
- net N$47: now also IC3A.QH*, IC7A.SER; no longer IC1A.QH*, IC2A.SER
- net N$48: now also IC2.RA3/MCLR#/VPP, ICSP.VPP/MCLR; no longer J1.VPP/MCLR, U$14.RA3/MCLR#/VPP
- net N$5: now also IC5.OUT, R16.2, RR17.2; no longer R5.2, R7.2, U$13.OUT
- net N$50: now also LED10.A, R1.2; no longer L3.A, R28.2
- net N$51: now also L1.1; no longer C7.2, IC4.VIN
- net N$6: now also IC5.FB, R18.2, RR17.1; no longer R5.1, R6.2, U$13.FB
- net N$7: now also R16.1; no longer R7.1
- net N$8: now also R21.1; no longer R15.1
- net N$9: now also R21.2; no longer R15.2
- net NSHDNA: now also IC2.RC4/TX, IC5.SHDN#; no longer U$13.SHDN#, U$14.RC4/TX
- net NSHDNB: now also IC1.SHDN#, IC2.RC3/SS#; no longer U$12.SHDN#, U$14.RC3/SS#
- net SH_CLK: now also IC2.RA4/SDO, IC3A.SCK, IC7A.SCK; no longer IC1A.SCK, IC2A.SCK, U$14.RA4/SDO
- net ST_CLK: now also IC2.RA5, IC3A.SCL, IC7A.SCL; no longer IC1A.SCL, IC2A.SCL, U$14.RA5
- net VCC: now also C2.2, C4.2, C5.1, C6.1, C9.+, IC1.VCC, IC2.VDD, IC3A.RCK, IC4P.VCC, IC5.VCC, IC6.VOUT, IC7A.RCK, IC7P.VCC, ICSP.VDD, R1.1, R14.2, R19.1; no longer C12.+, C2.1, C4.1, C5.2, C6.2, IC1A.RCK, IC1P.VCC, IC2A.RCK, IC2P.VCC, IC4.VOUT, J1.VDD, R16.1, R26.2, R28.1, U$12.VCC, U$13.VCC, U$14.VDD
Other:
- note added: "LED DRIVER"
- note added: "MIDI INPUT"
- note added: "SWITCH INPUTS"
- note added: "VIDEO MUX 1"
- note added: "VIDEO MUX 2"
- moved on the sheet: C1, C2, C3, C4, C5, C6, C7, C8, INA1, INA2, INA3, INA4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
