File: hardware/midi-vidi.sch (EAGLE design)
At the start: 82 parts, among them IC1 MAX4311SO14, IC2 PIC16F1825SO14, IC3 74HC595D, IC4 4051D, IC5 MAX4311SO14, IC6 REG1117, IC7 74HC595D, IC8 B1S

Commit message: Fix DRC issues - FINAL REV 1 PCB
Parts:
- renumbered OK1 to IC9
Changed lines of the file:
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@@
 <part name="R4" library="rcl" deviceset="R-EU_" device="R0805"/>
 <part name="C6" library="rcl" deviceset="C-EU" device="C0805"/>
-<part name="OK1" library="optocoupler" deviceset="6N138" device=""/>
+<part name="IC9" library="optocoupler" deviceset="6N138" device=""/>
 <part name="D1" library="jasons_stuff" deviceset="0805DIODE" device=""/>
 <part name="R21" library="rcl" deviceset="R-EU_" device="R0805"/>
@@
 <instance part="R4" gate="G$1" x="152.4" y="-50.8" rot="R180"/>
 <instance part="C6" gate="G$1" x="111.76" y="-88.9" rot="R90"/>
-<instance part="OK1" gate="G$1" x="-5.08" y="53.34"/>
+<instance part="IC9" gate="G$1" x="-5.08" y="53.34"/>
 <instance part="D1" gate="G$1" x="-17.78" y="55.88"/>
 <instance part="R21" gate="G$1" x="-25.4" y="58.42" rot="R180"/>
@@
 </segment>
 <segment>
-<pinref part="OK1" gate="G$1" pin="GND"/>
+<pinref part="IC9" gate="G$1" pin="GND"/>
 <wire x1="7.62" y1="48.26" x2="25.4" y2="48.26" width="0.1524" layer="91"/>
 <pinref part="R20" gate="G$1" pin="1"/>
@@
 </segment>
 <segment>
-<pinref part="OK1" gate="G$1" pin="VCC"/>
+<pinref part="IC9" gate="G$1" pin="VCC"/>
 <wire x1="7.62" y1="58.42" x2="27.94" y2="58.42" width="0.1524" layer="91"/>
 <pinref part="R19" gate="G$1" pin="1"/>
@@
 <net name="N$8" class="0">
 <segment>
-<pinref part="OK1" gate="G$1" pin="A"/>
+<pinref part="IC9" gate="G$1" pin="A"/>
 <pinref part="D1" gate="G$1" pin="P$2"/>
 <wire x1="-17.78" y1="56.388" x2="-17.78" y2="58.42" width="0.1524" layer="91"/>
@@
 <net name="N$18" class="0">
 <segment>
-<pinref part="OK1" gate="G$1" pin="C"/>
+<pinref part="IC9" gate="G$1" pin="C"/>
 <pinref part="D1" gate="G$1" pin="P$1"/>
 <wire x1="-17.78" y1="51.308" x2="-17.78" y2="48.26" width="0.1524" layer="91"/>
@@
 <net name="MIDI" class="0">
 <segment>
-<pinref part="OK1" gate="G$1" pin="VO"/>
+<pinref part="IC9" gate="G$1" pin="VO"/>
 <pinref part="R19" gate="G$1" pin="2"/>
 <wire x1="7.62" y1="53.34" x2="10.16" y2="53.34" width="0.1524" layer="91"/>
@@
 <net name="N$22" class="0">
 <segment>
-<pinref part="OK1" gate="G$1" pin="VB"/>
+<pinref part="IC9" gate="G$1" pin="VB"/>
 <pinref part="R20" gate="G$1" pin="2"/>
 <wire x1="7.62" y1="55.88" x2="12.7" y2="55.88" width="0.1524" layer="91"/>

Commit message: updates - working for rev2
Connections:
- net ST_CLK: now also IC3A.RCK, IC7A.RCK; no longer IC3A.SCL, IC7A.SCL
- net VCC: now also IC3A.SCL, IC7A.SCL; no longer IC3A.RCK, IC7A.RCK
Changed lines of the file:
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@@
 </segment>
 <segment>
-<pinref part="IC3" gate="A" pin="RCK"/>
-<wire x1="-142.24" y1="48.26" x2="-162.56" y2="48.26" width="0.1524" layer="91"/>
-<wire x1="-162.56" y1="48.26" x2="-162.56" y2="10.16" width="0.1524" layer="91"/>
-<pinref part="IC7" gate="A" pin="RCK"/>
-<wire x1="-162.56" y1="10.16" x2="-162.56" y2="7.62" width="0.1524" layer="91"/>
-<wire x1="-142.24" y1="10.16" x2="-162.56" y2="10.16" width="0.1524" layer="91"/>
-<junction x="-162.56" y="10.16"/>
+<wire x1="-162.56" y1="53.34" x2="-162.56" y2="15.24" width="0.1524" layer="91"/>
 <label x="-165.1" y="7.62" size="1.778" layer="95" rot="R270"/>
+<pinref part="IC3" gate="A" pin="SCL"/>
+<wire x1="-162.56" y1="15.24" x2="-162.56" y2="7.62" width="0.1524" layer="91"/>
+<wire x1="-142.24" y1="53.34" x2="-162.56" y2="53.34" width="0.1524" layer="91"/>
+<pinref part="IC7" gate="A" pin="SCL"/>
+<wire x1="-142.24" y1="15.24" x2="-162.56" y2="15.24" width="0.1524" layer="91"/>
+<junction x="-162.56" y="15.24"/>
 </segment>
 <segment>
@@
 <net name="ST_CLK" class="0">
 <segment>
-<pinref part="IC3" gate="A" pin="SCL"/>
-<wire x1="-142.24" y1="53.34" x2="-149.86" y2="53.34" width="0.1524" layer="91"/>
-<wire x1="-149.86" y1="53.34" x2="-149.86" y2="15.24" width="0.1524" layer="91"/>
-<pinref part="IC7" gate="A" pin="SCL"/>
-<wire x1="-149.86" y1="15.24" x2="-142.24" y2="15.24" width="0.1524" layer="91"/>
-<wire x1="-149.86" y1="53.34" x2="-149.86" y2="81.28" width="0.1524" layer="91"/>
-<junction x="-149.86" y="53.34"/>
+<wire x1="-149.86" y1="81.28" x2="-149.86" y2="48.26" width="0.1524" layer="91"/>
 <label x="-149.86" y="83.82" size="1.778" layer="95" rot="R270"/>
-</segment>
-<segment>
+<pinref part="IC7" gate="A" pin="RCK"/>
+<wire x1="-149.86" y1="48.26" x2="-149.86" y2="10.16" width="0.1524" layer="91"/>
+<wire x1="-142.24" y1="10.16" x2="-149.86" y2="10.16" width="0.1524" layer="91"/>
+<pinref part="IC3" gate="A" pin="RCK"/>
+<wire x1="-142.24" y1="48.26" x2="-149.86" y2="48.26" width="0.1524" layer="91"/>
+<junction x="-149.86" y="48.26"/>
+</segment>
+<segment>
